Commit message: working simulator

File: ur_description/urdf/common.gazebo.xacro (robot description, xacro)
@@ -1,9 +1,6 @@
 <?xml version="1.0"?>
 <robot xmlns:xacro="http://www.ros.org/wiki/xacro">
-  <gazebo>
-    <plugin name="ros_control" filename="libgazebo_ros_control.so">
-      <!--robotNamespace>/</robotNamespace-->
-      <!--robotSimType>gazebo_ros_control/DefaultRobotHWSim</robotSimType-->
-    </plugin>
+  <xacro:macro name="ur5_gazebo" params="prefix name">
+  </xacro:macro>
 <!--
     <plugin name="gazebo_ros_power_monitor_controller" filename="libgazebo_ros_power_monitor.so">
@@ -20,4 +17,3 @@
     </plugin>
 -->
-  </gazebo>
 </robot>

File: ur_description/urdf/ur.gazebo.xacro (robot description, xacro)
@@ -1,6 +1,39 @@
 <?xml version="1.0"?>
 <robot xmlns:xacro="http://www.ros.org/wiki/xacro">
-  <xacro:macro name="ur_arm_gazebo" params="prefix">
+  <xacro:macro name="ur_arm_gazebo" params="prefix name">
     <!-- nothing to do here at the moment -->
+    <gazebo>
+    <plugin name="${name}_ros_control" filename="libgazebo_ros_control.so">
+      <robotNamespace>${name}</robotNamespace>
+      <!--robotSimType>gazebo_ros_control/DefaultRobotHWSim</robotSimType-->
+    </plugin>
+</gazebo>
+    <gazebo reference="${prefix}base_link">
+      <gravity>true</gravity>
+    </gazebo>
+    <gazebo reference="${prefix}shoulder_link">
+      <gravity>true</gravity>
+    </gazebo>
+    <gazebo reference="${prefix}upper_arm_link">
+      <gravity>true</gravity>
+    </gazebo>
+    <gazebo reference="${prefix}forearm_link">
+      <gravity>true</gravity>
+    </gazebo>
+    <gazebo reference="${prefix}wrist_1_link">
+      <gravity>true</gravity>
+    </gazebo>
+    <gazebo reference="${prefix}wrist_2_link">
+      <gravity>true</gravity>
+    </gazebo>
+    <gazebo reference="${prefix}wrist_3_link">
+      <gravity>true</gravity>
+    </gazebo>
+  <gazebo reference="${prefix}ee_link">
+      <gravity>true</gravity>
+    </gazebo>
+     <gazebo reference="${prefix}tool0">
+      <gravity>true</gravity>
+    </gazebo>
   </xacro:macro>
 </robot>

File: ur_description/urdf/ur5.urdf.xacro (robot description, xacro)
@@ -1,5 +1,5 @@
 <?xml version="1.0"?>
 <robot xmlns:xacro="http://www.ros.org/wiki/xacro">
-  <xacro:include filename="$(find ur_description)/urdf/ur.transmission.xacro" />
+  <xacro:include filename="$(find ur_description)/urdf/ur.transmission_with_ns.xacro" />
   <xacro:include filename="$(find ur_description)/urdf/ur.gazebo.xacro" />
   <property name="pi" value="3.14159265" />
@@ -186,8 +186,10 @@
       <axis xyz="0 1 0" />
       <xacro:unless value="${joint_limited}">
-        <limit lower="${-2.0 * pi}" upper="${2.0 * pi}" effort="28.0" velocity="3.2"/>
-      </xacro:unless>
-      <xacro:if value="${joint_limited}">
-        <limit lower="${-pi}" upper="${pi}" effort="28.0" velocity="3.2"/>
+        <limit lower="${-2.0 * pi}" upper="${2.0 * pi}" effort="28.0" acceleration="1.0" velocity="3.2"/>
+        <!--safety_controller k_position="5.0"  k_velocity="0.5" /-->
+      </xacro:unless>
+      <xacro:if value="${joint_limited}">
+        <limit lower="${-pi}" upper="${pi}" effort="28.0" acceleration="1.0" velocity="3.2"/>
+        <!--safety_controller k_position="5.0"  k_velocity="0.5" /-->
       </xacro:if>
       <dynamics damping="0.0" friction="0.0"/>
@@ -217,8 +219,10 @@
       <axis xyz="0 0 1" />
       <xacro:unless value="${joint_limited}">
-        <limit lower="${-2.0 * pi}" upper="${2.0 * pi}" effort="28.0" velocity="3.2"/>
-      </xacro:unless>
-      <xacro:if value="${joint_limited}">
-        <limit lower="${-pi}" upper="${pi}" effort="28.0" velocity="3.2"/>
+        <limit lower="${-2.0 * pi}" upper="${2.0 * pi}" effort="28.0" acceleration="1.0" velocity="3.2"/>
+        <!--safety_controller k_position="5.0"  k_velocity="0.5" /-->
+      </xacro:unless>
+      <xacro:if value="${joint_limited}">
+        <limit lower="${-pi}" upper="${pi}" effort="28.0" acceleration="1.0" velocity="3.2"/>
+        <!--safety_controller k_position="5.0"  k_velocity="0.5" /-->
       </xacro:if>
       <dynamics damping="0.0" friction="0.0"/>
@@ -248,8 +252,10 @@
       <axis xyz="0 1 0" />
       <xacro:unless value="${joint_limited}">
-        <limit lower="${-2.0 * pi}" upper="${2.0 * pi}" effort="28.0" velocity="3.2"/>
-      </xacro:unless>
-      <xacro:if value="${joint_limited}">
-        <limit lower="${-pi}" upper="${pi}" effort="28.0" velocity="3.2"/>
+        <limit lower="${-2.0 * pi}" upper="${2.0 * pi}" effort="28.0" acceleration="1.0" velocity="3.2"/>
+        <!--safety_controller k_position="5.0"  k_velocity="0.5" /-->
+      </xacro:unless>
+      <xacro:if value="${joint_limited}">
+        <limit lower="${-pi}" upper="${pi}" effort="28.0" acceleration="1.0" velocity="3.2"/>
+        <!--safety_controller k_position="5.0"  k_velocity="0.5" /-->
       </xacro:if>
       <dynamics damping="0.0" friction="0.0"/>
@@ -286,6 +292,6 @@
       </collision>
     </link>
-    <xacro:ur_arm_transmission prefix="${prefix}" />
-    <xacro:ur_arm_gazebo prefix="${prefix}" />
+    <xacro:ur_arm_transmission prefix="${prefix}" name="ur5" />
+    <xacro:ur_arm_gazebo prefix="${prefix}" name="ur5"/>
     <!-- ROS base_link to UR 'Base' Coordinates transform -->
     <link name="${prefix}base"/>
